Commit message: modified lite3 training

File: resources/deepRobotics/lite3/urdf/Lite3.urdf (robot description, URDF)
Before this commit: robot Lite3, 17 links, 16 joints
Links:
- added link INERTIA, mass 4.130
- link FL_FOOT: geometry collision sphere radius=0.013
- link FL_HIP: mass 0.550 -> 0.428; geometry visual mesh filename=../meshes/FL_HIP.dae
- link FL_SHANK: mass 0.153 -> 0.115; geometry collision box size=0.02 0.02 0.18; visual mesh filename=../meshes/SHANK.dae
- link FL_THIGH: mass 0.86 -> 0.61; geometry collision box size=0.02 0.02 0.16; visual mesh filename=../meshes/L_THIGH.dae
- link FR_FOOT: geometry collision sphere radius=0.013
- link FR_HIP: mass 0.550 -> 0.428; geometry visual mesh filename=../meshes/FR_HIP.dae
- link FR_SHANK: mass 0.153 -> 0.115; geometry collision box size=0.02 0.02 0.18; visual mesh filename=../meshes/SHANK.dae
- link FR_THIGH: mass 0.86 -> 0.61; geometry collision box size=0.02 0.02 0.16; visual mesh filename=../meshes/R_THIGH.dae
- link HL_FOOT: geometry collision sphere radius=0.013
- link HL_HIP: mass 0.550 -> 0.428; geometry visual mesh filename=../meshes/HL_HIP.dae
- link HL_SHANK: mass 0.153 -> 0.115; geometry collision box size=0.02 0.02 0.18; visual mesh filename=../meshes/SHANK.dae
- link HL_THIGH: mass 0.86 -> 0.61; geometry collision box size=0.02 0.02 0.16; visual mesh filename=../meshes/L_THIGH.dae
- link HR_FOOT: geometry collision sphere radius=0.013
- link HR_HIP: mass 0.550 -> 0.428; geometry visual mesh filename=../meshes/HR_HIP.dae
- link HR_SHANK: mass 0.153 -> 0.115; geometry collision box size=0.02 0.02 0.18; visual mesh filename=../meshes/SHANK.dae
- link HR_THIGH: mass 0.86 -> 0.61; geometry collision box size=0.02 0.02 0.16; visual mesh filename=../meshes/R_THIGH.dae
- link TORSO: mass 5.6056 -> None; geometry collision box size=0.35 0.184 0.08; visual mesh filename=../meshes/Lite3.dae
Joints:
- added joint Torso2Inertia: type fixed, parent TORSO, child INERTIA
- joint FL_Ankle: origin xyz=0 0 -0.21012 -> xyz=0 0 -0.21
- joint FL_HipX_joint: limit lower=-0.523 upper=0.523 effort=30 velocity=20 -> lower=-0.42 upper=0.42 effort=24 velocity=26; origin xyz=0.1745 0.062 0 rpy=0 0 0 -> xyz=0.1745 0.062 0
- joint FL_HipY_joint: limit lower=-2.67 upper=0.314 effort=30 velocity=20 -> lower=-2.67 upper=0.314 effort=24 velocity=26; origin xyz=0 0.09735 0 rpy=0 0 0 -> xyz=0 0.0985 0
- joint FL_Knee_joint: limit lower=0.524 upper=2.792 effort=30 velocity=20 -> lower=0.6 upper=2.72 effort=36 velocity=17; origin xyz=0 0 -0.20 rpy=0 0 0 -> xyz=0 0 -0.20
- joint FR_Ankle: origin xyz=0 0 -0.21012 -> xyz=0 0 -0.21
- joint FR_HipX_joint: limit lower=-0.523 upper=0.523 effort=30 velocity=20 -> lower=-0.42 upper=0.42 effort=24 velocity=26; origin xyz=0.1745 -0.062 0 rpy=0 0 0 -> xyz=0.1745 -0.062 0
- joint FR_HipY_joint: limit lower=-2.67 upper=0.314 effort=30 velocity=20 -> lower=-2.67 upper=0.314 effort=24 velocity=26; origin xyz=0 -0.09735 0 rpy=0 0 0 -> xyz=0 -0.0985 0
- joint FR_Knee_joint: limit lower=0.524 upper=2.792 effort=30 velocity=20 -> lower=0.6 upper=2.72 effort=36 velocity=17; origin xyz=0 0 -0.20 rpy=0 0 0 -> xyz=0 0 -0.20
- joint HL_Ankle: origin xyz=0 0 -0.21012 -> xyz=0 0 -0.21
- joint HL_HipX_joint: limit lower=-0.523 upper=0.523 effort=30 velocity=20 -> lower=-0.42 upper=0.42 effort=24 velocity=26; origin xyz=-0.1745 0.062 0 rpy=0 0 0 -> xyz=-0.1745 0.062 0
- joint HL_HipY_joint: limit lower=-2.67 upper=0.314 effort=30 velocity=20 -> lower=-2.67 upper=0.314 effort=24 velocity=26; origin xyz=0 0.09735 0 rpy=0 0 0 -> xyz=0 0.0985 0
- joint HL_Knee_joint: limit lower=0.524 upper=2.792 effort=30 velocity=20 -> lower=0.6 upper=2.72 effort=36 velocity=17; origin xyz=0 0 -0.20 rpy=0 0 0 -> xyz=0 0 -0.20
- joint HR_Ankle: origin xyz=0 0 -0.21012 -> xyz=0 0 -0.21
- joint HR_HipX_joint: limit lower=-0.523 upper=0.523 effort=30 velocity=20 -> lower=-0.42 upper=0.42 effort=24 velocity=26; origin xyz=-0.1745 -0.062 0 rpy=0 0 0 -> xyz=-0.1745 -0.062 0
- joint HR_HipY_joint: limit lower=-2.67 upper=0.314 effort=30 velocity=20 -> lower=-2.67 upper=0.314 effort=24 velocity=26; origin xyz=0 -0.09735 0 rpy=0 0 0 -> xyz=0 -0.0985 0
- joint HR_Knee_joint: limit lower=0.524 upper=2.792 effort=30 velocity=20 -> lower=0.6 upper=2.72 effort=36 velocity=17; origin xyz=0 0 -0.20 rpy=0 0 0 -> xyz=0 0 -0.20
